File: TZXDUINO.brd (EAGLE design)
At the start: 6.2 x 10.8 mm, 20 parts, among them IC1 LM386N-1, J1 DCJ0202, J2 JW-PJ-307-5, X1 1501_04

Commit message: Add files via upload
Routing:
- net N$24: track 0.00 -> 2.25 mm
Changed lines of the file:
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@@
 <layer number="21" name="tPlace" color="7" fill="1" visible="yes" active="yes"/>
 <layer number="22" name="bPlace" color="7" fill="1" visible="yes" active="yes"/>
-<layer number="23" name="tOrigins" color="15" fill="1" visible="no" active="yes"/>
+<layer number="23" name="tOrigins" color="15" fill="1" visible="yes" active="yes"/>
 <layer number="24" name="bOrigins" color="15" fill="1" visible="yes" active="yes"/>
 <layer number="25" name="tNames" color="7" fill="1" visible="yes" active="yes"/>
@@
 <layer number="42" name="bRestrict" color="1" fill="10" visible="yes" active="yes"/>
 <layer number="43" name="vRestrict" color="2" fill="10" visible="yes" active="yes"/>
-<layer number="44" name="Drills" color="7" fill="1" visible="no" active="yes"/>
-<layer number="45" name="Holes" color="7" fill="1" visible="no" active="yes"/>
+<layer number="44" name="Drills" color="7" fill="1" visible="yes" active="yes"/>
+<layer number="45" name="Holes" color="7" fill="1" visible="yes" active="yes"/>
 <layer number="46" name="Milling" color="3" fill="1" visible="yes" active="yes"/>
 <layer number="47" name="Measures" color="7" fill="1" visible="yes" active="yes"/>
@@
 <layer number="131" name="tAdjust" color="7" fill="1" visible="no" active="no"/>
 <layer number="132" name="bAdjust" color="7" fill="1" visible="no" active="no"/>
-<layer number="144" name="DrillLegend" color="7" fill="1" visible="no" active="yes"/>
-<layer number="145" name="DrillLegend_01-16" color="2" fill="9" visible="no" active="yes"/>
-<layer number="146" name="DrillLegend_01-20" color="3" fill="9" visible="no" active="yes"/>
+<layer number="144" name="DrillLegend" color="7" fill="1" visible="yes" active="yes"/>
+<layer number="145" name="DrillLegend_01-16" color="2" fill="9" visible="yes" active="yes"/>
+<layer number="146" name="DrillLegend_01-20" color="3" fill="9" visible="yes" active="yes"/>
 <layer number="150" name="Notes" color="7" fill="1" visible="no" active="no"/>
 <layer number="151" name="HeatSink" color="7" fill="1" visible="no" active="no"/>
@@
 <wire x1="29" y1="38.275" x2="28.492" y2="38.783" width="0.1016" layer="146"/>
 <wire x1="29" y1="38.275" x2="29" y2="37.767" width="0.1016" layer="146"/>
+<circle x="6.4027" y="13.8496" radius="1.67705" width="0.127" layer="21"/>
+<circle x="5.6527" y="14.6671" radius="0.25" width="0.127" layer="21"/>
+<circle x="7.1527" y="14.6671" radius="0.25" width="0.127" layer="21"/>
+<circle x="6.4027" y="13.5996" radius="0.25" width="0.127" layer="21"/>
+<wire x1="7.5277" y1="13.4746" x2="5.2777" y2="13.5996" width="0.127" layer="21" curve="-161.131001"/>
+<circle x="13.6777" y="53.1496" radius="1.67705" width="0.127" layer="16"/>
+<circle x="12.9277" y="53.9671" radius="0.25" width="0.127" layer="16"/>
+<circle x="14.4277" y="53.9671" radius="0.25" width="0.127" layer="16"/>
+<circle x="13.6777" y="52.8996" radius="0.25" width="0.127" layer="16"/>
 </plain>
 <attributes>
@@
 </element>
 <element name="U$1" library="diy-modules" package="DISPLAY-OLED-128X64-I2C" value="DISPLAY-OLED-128X64-I2C" x="38.8325" y="54.8875" smashed="yes">
-<attribute name="VALUE" x="38.8325" y="39.6475" size="1.27" layer="27" align="top-center"/>
+<attribute name="VALUE" x="38.8325" y="39.6475" size="1.27" layer="25" align="top-center"/>
 </element>
 <element name="U1" library="RGU-StoresParts" package="ARDUINO_NANO" value="" x="53.12" y="25.36" smashed="yes">
@@
 <attribute name="NAME" x="65.4665" y="41.3415" size="1.27" layer="25" ratio="10"/>
 <attribute name="POPULARITY" value="0" x="66.2125" y="48.3825" size="1.778" layer="27" rot="R270" display="off"/>
-<attribute name="VALUE" x="65.5775" y="51.9385" size="1.27" layer="27" ratio="10" rot="R270"/>
+<attribute name="VALUE" x="65.5775" y="51.9385" size="1.27" layer="25" ratio="10" rot="R270"/>
 </element>
 <element name="C1" library="RGU-StoresParts" package="E3,5-8" value="220uF" x="74.3925" y="63.7775" smashed="yes">
 <attribute name="NAME" x="73.1945" y="65.8215" size="1.27" layer="25" ratio="10"/>
-<attribute name="VALUE" x="72.3315" y="60.8795" size="1.27" layer="27" ratio="10"/>
+<attribute name="VALUE" x="72.3315" y="60.8795" size="1.27" layer="25" ratio="10"/>
 </element>
 <element name="C2" library="RGU-StoresParts" package="C050-025X075" value="100nF" x="64.8675" y="57.745" smashed="yes" rot="R180">
 <attribute name="NAME" x="62.7465" y="56.094" size="1.27" layer="25" ratio="10" rot="R180"/>
-<attribute name="VALUE" x="68.1465" y="56.114" size="1.27" layer="27" ratio="10" rot="R180"/>
+<attribute name="VALUE" x="68.1465" y="56.114" size="1.27" layer="25" ratio="10" rot="R180"/>
 </element>
 <element name="C4" library="RGU-StoresParts" package="C050-025X075" value="47nF" x="73.1225" y="57.745" smashed="yes">
 <attribute name="NAME" x="70.6685" y="54.746" size="1.27" layer="25" ratio="10"/>
-<attribute name="VALUE" x="73.3685" y="54.801" size="1.27" layer="27" ratio="10"/>
+<attribute name="VALUE" x="73.3685" y="54.801" size="1.27" layer="25" ratio="10"/>
 </element>
 <element name="R1" library="RGU-StoresParts" package="0207/10" value="10r" x="75.68" y="44.4875" smashed="yes" rot="R90">
 <attribute name="NAME" x="76.7605" y="37.556" size="1.27" layer="25" ratio="10" rot="R180"/>
-<attribute name="VALUE" x="76.315" y="42.9769" size="1.27" layer="27" ratio="10" rot="R90"/>
+<attribute name="VALUE" x="76.315" y="42.9769" size="1.27" layer="25" ratio="10" rot="R90"/>
 </element>
 <element name="C5" library="RGU-StoresParts" package="E2,5-5" value="10uF" x="57.565" y="63.7775" smashed="yes">
 <attribute name="NAME" x="56.828" y="66.8475" size="1.27" layer="25" ratio="10"/>
-<attribute name="VALUE" x="55.853" y="59.4895" size="1.27" layer="27" ratio="10"/>
+<attribute name="VALUE" x="55.853" y="59.4895" size="1.27" layer="25" ratio="10"/>
 </element>
 <element name="C6" library="RGU-StoresParts" package="E2,5-5" value="100uF" x="65.185" y="63.7775" smashed="yes">
 <attribute name="NAME" x="64.448" y="66.6975" size="1.27" layer="25" ratio="10"/>
-<attribute name="VALUE" x="62.723" y="59.7145" size="1.27" layer="27" ratio="10"/>
+<attribute name="VALUE" x="62.723" y="59.7145" size="1.27" layer="25" ratio="10"/>
 </element>
 <element name="DRILEGEND" library="drilegend" package="DRILEGEND" value="" x="-4.82000625" y="-3.88500625" smashed="yes"/>
@@
 <via x="81.3" y="34.05" extent="1-16" drill="0.8"/>
 </signal>
+<signal name="N$24">
+<wire x1="14.8027" y1="52.7746" x2="12.5527" y2="52.8996" width="0.127" layer="16" curve="-161.131001"/>
+</signal>
 </signals>
